File: PCB_design.kicad_sch (KiCad schematic)
At the start: 30 parts, among them J1 Conn_02x05_Odd_Even, J2 Conn_02x03_Odd_Even, Q1 Q_NMOS_DGS, SW3 SW_Push, U1 LT1117-ADJ, U2 STM32F091RCTx, Y1 Crystal_GND24, Y2 Crystal_GND24

Commit message: Add files via upload
Parts:
- removed C15, C16: 20pF, symbol Device:C
- removed C9: 100n, symbol Device:C
- removed J1: Conn_02x05_Odd_Even, symbol Connector_Generic:Conn_02x05_Odd_Even
- removed Y1, Y2: Crystal_GND24, symbol Device:Crystal_GND24
- added C? (x2): 20pF, symbol Device:C
- added R?: 390, symbol Device:R
- added Y?: Crystal, symbol Device:Crystal
Connections:
- net GND: now also C?.2, C?.2
- net at J2.5 (Pin_5): now also C?.1, Y?.1
- net at J2.6 (Pin_6): now also R?.2
- new net: C?.1, R?.1, Y?.2
- no-connect marks 1 -> 0
Other:
- moved on the sheet: J2

Commit message: Add files via upload
Parts:
- removed C10: 500, symbol Device:C
- removed C11: 160p, symbol Device:C
- removed C12: 100u, symbol Device:C
- removed C13: C, symbol Device:C
- removed C14: 10u, symbol Device:C
- removed C? (x2): 20pF, symbol Device:C
- removed D1: 1N5819, Diode_THT:D_DO-41_SOD81_P10.16mm_Horizontal, symbol Diode:1N5819
- removed L1: 50, symbol Device:L
- removed Q1: Q_NMOS_DGS, symbol Device:Q_NMOS_DGS
- removed R1: 50, symbol Device:R
- removed R2: 200, symbol Device:R
- removed R3: 120, symbol Device:R
- removed R?: 390, symbol Device:R
- removed U1: LT1117-ADJ, symbol Regulator_Linear:LT1117-ADJ
- removed Y?: Crystal, symbol Device:Crystal
- added C?: 20pF, symbol Device:C
- added D?: D, symbol Device:D
- added J?: Conn_02x05_Odd_Even, symbol Connector_Generic:Conn_02x05_Odd_Even
- added R?: 5.1k, symbol Device:R
- added U?: MAX7375AXR805, Package_TO_SOT_SMD:SOT-323_SC-70, symbol Oscillator:MAX7375AXR805
Connections:
- net GND is gone; now on net +3.3VA: C1.2, C17.2, C18.2, C19.2, C20.2, C21.2, R5.1, SW3.1, U2.12 (VSSA), U2.18 (VSS), U2.31 (VSS), U2.47 (VSS), U2.63 (VSS)
- net +3.3V: now also C?.1, U?.1 (V+)
- net +3.3VA: now also C?.2, D?.1 (K), D?.2 (A), J?.10 (Pin_10), J?.3 (Pin_3), J?.4 (Pin_4), J?.9 (Pin_9), R?.1, R?.2, U?.3 (GND)
- net NRST: now also J?.1 (Pin_1)
- net at J2.6 (Pin_6): now also J2.5 (Pin_5), U?.2 (CLOCK)
- net BOOT0 PF11 renamed BOOT0_PF11
- net PA13 renamed PA13 SWDIO_IN
- net PA13 SWDIO_IN: now also J?.2 (Pin_2)
- net PA14 renamed PA14 SWCLK_IN
- net PA14 SWCLK_IN: now also J?.6 (Pin_6)
- new net V3.3_IN: J?.7 (Pin_7), J?.8 (Pin_8)
- no-connect marks 0 -> 1
Other:
- added sheet Page 2 (PCB_design2.kicad_sch)
- note added: "Decoupling Capacitors and Filter"
- note added: "General Purpose Timer"
- note added: "Programming Header"
- note added: "Reset Circuit"
- note removed: "5V to 3.3V LDO"
- note removed: "NMOS Motor Driver"
- moved on the sheet: J2
